Commit message: [rjjt] added pi camera to model

File: src/arduinobot_description/urdf/arduinobot.urdf.xacro (robot description, xacro)
@@ -117,3 +117,19 @@
       velocity="${velocity}" />
   </joint>
+  <link name="rgb_camera">
+    <visual>
+      <origin xyz="-0.135 0.125 0" rpy="0 0 -${PI/2}" />
+      <geometry>
+        <mesh filename="package://arduinobot_description/meshes/pi_camera.STL"
+          scale="0.01 0.01 0.01" />
+      </geometry>
+    </visual>
+  </link>
+  <joint name="rgb_camera_joint" type="revolute">
+    <parent link="base_link" />
+    <child link="rgb_camera" />
+    <axis xyz="0 1 0" />
+    <origin rpy="0 -0.5 1.57" xyz="0 0.45 0.2" />
+    <limit lower="${PI/2}" upper="${PI*3/4}" effort="${effort}" velocity="${velocity}" />
+  </joint>
 </robot>

Commit message: [rjjt] added controller

File: src/arduinobot_description/urdf/arduinobot.urdf.xacro (robot description, xacro)
@@ -1,9 +1,21 @@
 <?xml version="1.0"?>
 <robot xmlns:xacro="http://www.ros.org/wiki/xacro" name="arduinobot">
+  <xacro:arg name="is_ignition" default="true" />
+  <xacro:include filename="$(find arduinobot_description)/urdf/arduinobot_gazebo.xacro" />
+  <xacro:include filename="$(find arduinobot_description)/urdf/arduinobot_ros2_control.xacro" />
   <xacro:property name="PI" value="3.14159" />
   <xacro:property name="effort" value="30.0" />
   <xacro:property name="velocity" value="10.0" />
+  <xacro:macro name="default_inertial" params="mass">
+    <inertial>
+      <mass value="${mass}" />
+      <inertia ixx="1.0" ixy="0.0" ixz="0.0"
+        iyy="1.0" iyz="0.0"
+        izz="1.0" />
+    </inertial>
+  </xacro:macro>
   <link name="world" />
   <link name="base_link">
+    <xacro:default_inertial mass="1.0" />
     <visual>
       <origin rpy="0 0 0" xyz="-0.5 -0.5 0" />
@@ -12,4 +24,10 @@
       </geometry>
     </visual>
+    <collision>
+      <origin rpy="0 0 0" xyz="-0.5 -0.5 0" />
+      <geometry>
+        <mesh filename="package://arduinobot_description/meshes/basement.STL" scale="0.01 0.01 0.01" />
+      </geometry>
+    </collision>
   </link>
   <joint name="virtual_joint" type="fixed">
@@ -19,4 +37,5 @@
   </joint>
   <link name="base_plate">
+    <xacro:default_inertial mass="0.1" />
     <visual>
       <origin rpy="0 0 0" xyz="-0.39 -0.39 -0.56" />
@@ -26,4 +45,11 @@
       </geometry>
     </visual>
+    <collision>
+      <origin rpy="0 0 0" xyz="-0.39 -0.39 -0.56" />
+      <geometry>
+        <mesh filename="package://arduinobot_description/meshes/base_plate.STL"
+          scale="0.01 0.01 0.01" />
+      </geometry>
+    </collision>
   </link>
   <joint name="joint_1" type="revolute">
@@ -35,4 +61,5 @@
   </joint>
   <link name="forward_drive_arm">
+    <xacro:default_inertial mass="0.1" />
     <visual>
       <origin rpy="0 -${PI/2} ${PI/2}" xyz="0.19 0.06 -0.08" />
@@ -42,4 +69,11 @@
       </geometry>
     </visual>
+    <collision>
+      <origin rpy="0 -${PI/2} ${PI/2}" xyz="0.19 0.06 -0.08" />
+      <geometry>
+        <mesh filename="package://arduinobot_description/meshes/forward_drive_arm.STL"
+          scale="0.01 0.01 0.01" />
+      </geometry>
+    </collision>
   </link>
   <joint name="joint_2" type="revolute">
@@ -51,4 +85,5 @@
   </joint>
   <link name="horizontal_arm">
+    <xacro:default_inertial mass="0.1" />
     <visual>
       <origin rpy="${PI/2} 0 ${PI/2}" xyz="-0.03 -0.4 -0.06" />
@@ -58,4 +93,11 @@
       </geometry>
     </visual>
+    <collision>
+      <origin rpy="${PI/2} 0 ${PI/2}" xyz="-0.03 -0.4 -0.06" />
+      <geometry>
+        <mesh filename="package://arduinobot_description/meshes/horizontal_arm.STL"
+          scale="0.01 0.01 0.01" />
+      </geometry>
+    </collision>
   </link>
   <joint name="joint_3" type="revolute">
@@ -68,4 +110,5 @@
       velocity="${velocity}" /> w </joint>
   <link name="claw_support">
+    <xacro:default_inertial mass="0.05" />
     <visual>
       <origin rpy="0 0 ${PI/2}" xyz="0 -0.05 -0.15" />
@@ -75,4 +118,11 @@
       </geometry>
     </visual>
+    <collision>
+      <origin rpy="0 0 ${PI/2}" xyz="0 -0.05 -0.15" />
+      <geometry>
+        <mesh filename="package://arduinobot_description/meshes/claw_support.STL"
+          scale="0.01 0.01 0.01" />
+      </geometry>
+    </collision>
   </link>
   <joint name="horizontal_arm_to_claw_support" type="fixed">
@@ -82,4 +132,5 @@
   </joint>
   <link name="gripper_right">
+    <xacro:default_inertial mass="0.01" />
     <visual>
       <origin xyz="-0.1 0.5 -0.1" rpy="0 0 -${PI/2}" />
@@ -89,6 +140,14 @@
       </geometry>
     </visual>
+    <collision>
+      <origin xyz="-0.1 0.5 -0.1" rpy="0 0 -${PI/2}" />
+      <geometry>
+        <mesh filename="package://arduinobot_description/meshes/right_finger.STL"
+          scale="0.01 0.01 0.01" />
+      </geometry>
+    </collision>
   </link>
   <link name="gripper_left">
+    <xacro:default_inertial mass="0.01" />
     <visual>
       <origin xyz="-0.04 0.5 -0.1" rpy="0 0 -${PI/2}" />
@@ -98,4 +157,11 @@
       </geometry>
     </visual>
+    <collision>
+      <origin xyz="-0.04 0.5 -0.1" rpy="0 0 -${PI/2}" />
+      <geometry>
+        <mesh filename="package://arduinobot_description/meshes/left_finger.STL"
+          scale="0.01 0.01 0.01" />
+      </geometry>
+    </collision>
   </link>
   <joint name="joint_4" type="revolute">
@@ -118,6 +184,7 @@
   </joint>
   <link name="rgb_camera">
-    <visual>
-      <origin xyz="-0.135 0.125 0" rpy="0 0 -${PI/2}" />
+    <xacro:default_inertial mass="0.001" />
+    <visual>
+      <origin rpy="-1.57 0 -1.57" xyz="-0.1 0.125 0.15" />
       <geometry>
         <mesh filename="package://arduinobot_description/meshes/pi_camera.STL"
@@ -125,11 +192,47 @@
       </geometry>
     </visual>
-  </link>
-  <joint name="rgb_camera_joint" type="revolute">
+    <collision>
+      <origin rpy="-1.57 0 -1.57" xyz="-0.1 0.125 0.15" />
+      <geometry>
+        <mesh filename="package://arduinobot_description/meshes/pi_camera.STL"
+          scale="0.01 0.01 0.01" />
+      </geometry>
+    </collision>
+  </link>
+  <joint name="rgb_camera_joint" type="fixed">
     <parent link="base_link" />
     <child link="rgb_camera" />
     <axis xyz="0 1 0" />
     <origin rpy="0 -0.5 1.57" xyz="0 0.45 0.2" />
-    <limit lower="${PI/2}" upper="${PI*3/4}" effort="${effort}" velocity="${velocity}" />
-  </joint>
+  </joint>
+  <gazebo reference="rgb_camera">
+    <sensor name="camera" type="camera">
+      <always_on>true</always_on>
+      <update_rate>30.0</update_rate>
+      <visualize>true</visualize>
+      <topic>/image_raw</topic>
+      <gz_frame_id>/rgb_camera</gz_frame_id>
+      <camera name="camera">
+        <horizontal_fov>1.21126</horizontal_fov>
+        <image>
+          <width>2304</width>
+          <height>1296</height>
+          <format>R8G8B8</format>
+        </image>
+        <distortion>
+          <k1>0.0</k1>
+          <k2>0.0</k2>
+          <k3>0.0</k3>
+          <p1>0.0</p1>
+          <p2>0.0</p2>
+          <center>0.5 0.5</center>
+        </distortion>
+      </camera>
+    </sensor>
+  </gazebo>
+  <gazebo>
+    <plugin name="camera_controller" filename="libgazebo_ros_camera.so">
+      <frame_name>rgb_camera</frame_name>
+    </plugin>
+  </gazebo>
 </robot>
